File: PCB/ArduinoUnoCape/ArduinoCape.brd (EAGLE design)
At the start: 160 x 100 mm, 1 part, among them U1 ARDUINOR3-DIMENSION

Commit message: updated pcb and code
Parts:
- added 7-SEG-LED: 4P-2.0, Seeed-OPL-Connector:HW4-2.0
- added BUTTON: (no value), pinhead:1X02
- added J1: (no value), SparkFun-Connectors:JST-2-PTH
- added LED: (no value), con-lstb:MA03-1
- moved U1 81.3 mm to (0.00, 0.00)
Connections:
- net 3V renamed 3V3
- net 5V: now also 7-SEG-LED.3
- net BUTTON: now also BUTTON.2
- net GND: now also 7-SEG-LED.4, BUTTON.1, J1.1
- net GREEN: now also LED.1
- net RED: now also LED.3
- net SCL: now also 7-SEG-LED.1, U1.SCL; no longer U1.A5
- net SDA: now also 7-SEG-LED.2, U1.SDA; no longer U1.A4
- net VIN: now also J1.2
- net YELLOW: now also LED.2
Routing:
- net VIN: track 0.00 -> 53.8 mm, vias 0 -> 1
- net SCL: track 0.00 -> 30.5 mm
- net SDA: track 0.00 -> 30.3 mm
- net 5V: track 0.00 -> 24.1 mm
- net BUTTON: track 0.00 -> 18.4 mm
- net GND: track 0.00 -> 8.57 mm
- net YELLOW: track 0.00 -> 7.62 mm
- net RED: track 0.00 -> 7.62 mm
- net GREEN: track 0.00 -> 7.62 mm
- added copper zone on layer 16, net GND
Other:
- board size 160 x 100 mm -> 68.6 x 53.3 mm

Commit message: asdf
Parts:
- 7-SEG-LED: value 4P-2.0 -> (none)
- moved LED 6.98 mm to (53.3, 36.2)
- moved BUTTON 6.25 mm to (54.6, 26.7)
- renumbered J1 to BATERRY
Routing:
- net YELLOW: track 7.62 -> 14.6 mm
- net RED: track 7.62 -> 14.6 mm
- net GREEN: track 7.62 -> 14.6 mm
- net BUTTON: track 18.4 -> 25.2 mm
Changed lines of the file:
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@@
 </autorouter>
 <elements>
-<element name="7-SEG-LED" library="Seeed-OPL-Connector" package="HW4-2.0" value="4P-2.0" x="31.115" y="24.13"/>
-<element name="J1" library="SparkFun-Connectors" package="JST-2-PTH" value="" x="6.35" y="24.13" rot="R90">
+<element name="7-SEG-LED" library="Seeed-OPL-Connector" package="HW4-2.0" value="" x="31.115" y="24.13"/>
+<element name="BATERRY" library="SparkFun-Connectors" package="JST-2-PTH" value="" x="6.35" y="24.13" rot="R90">
 <attribute name="PROD_ID" value="CONN-09863" x="6.35" y="24.13" size="1.778" layer="27" rot="R90" display="off"/>
 <attribute name="SKU" value="PRT-09914" x="6.35" y="24.13" size="1.778" layer="27" rot="R90" display="off"/>
 </element>
-<element name="LED" library="con-lstb" library_urn="urn:adsk.eagle:library:162" package="MA03-1" value="" x="53.34" y="43.18" rot="R180">
-<attribute name="MF" value="" x="53.34" y="43.18" size="1.778" layer="27" rot="R180" display="off"/>
-<attribute name="MPN" value="" x="53.34" y="43.18" size="1.778" layer="27" rot="R180" display="off"/>
-<attribute name="OC_FARNELL" value="unknown" x="53.34" y="43.18" size="1.778" layer="27" rot="R180" display="off"/>
-<attribute name="OC_NEWARK" value="unknown" x="53.34" y="43.18" size="1.778" layer="27" rot="R180" display="off"/>
+<element name="LED" library="con-lstb" library_urn="urn:adsk.eagle:library:162" package="MA03-1" value="" x="53.34" y="36.195" rot="R180">
+<attribute name="MF" value="" x="53.34" y="36.195" size="1.778" layer="27" rot="R180" display="off"/>
+<attribute name="MPN" value="" x="53.34" y="36.195" size="1.778" layer="27" rot="R180" display="off"/>
+<attribute name="OC_FARNELL" value="unknown" x="53.34" y="36.195" size="1.778" layer="27" rot="R180" display="off"/>
+<attribute name="OC_NEWARK" value="unknown" x="53.34" y="36.195" size="1.778" layer="27" rot="R180" display="off"/>
 </element>
 <element name="U1" library="adafruit" library_urn="urn:adsk.eagle:library:420" package="ARDUINOR3" value="ARDUINOR3-DIMENSION" x="0" y="0" smashed="yes"/>
-<element name="BUTTON" library="pinhead" library_urn="urn:adsk.eagle:library:325" package="1X02" value="" x="57.15" y="32.385"/>
+<element name="BUTTON" library="pinhead" library_urn="urn:adsk.eagle:library:325" package="1X02" value="" x="54.61" y="26.67"/>
 </elements>
 <signals>
@@
 <contactref element="U1" pad="GND1"/>
 <contactref element="7-SEG-LED" pad="4"/>
-<contactref element="J1" pad="1"/>
+<contactref element="BATERRY" pad="1"/>
 <contactref element="BUTTON" pad="1"/>
 <wire x1="6.35" y1="23.13" x2="7.35" y2="23.13" width="0.508" layer="1"/>
@@
 <contactref element="U1" pad="D2"/>
 <contactref element="BUTTON" pad="2"/>
-<wire x1="58.42" y1="50.8" x2="58.42" y2="32.385" width="0.3048" layer="16"/>
+<wire x1="58.42" y1="29.21" x2="55.88" y2="26.67" width="0.3048" layer="16"/>
+<wire x1="58.42" y1="50.8" x2="58.42" y2="29.21" width="0.3048" layer="16"/>
 </signal>
 <signal name="GREEN">
 <contactref element="U1" pad="D3"/>
 <contactref element="LED" pad="1"/>
-<wire x1="55.88" y1="50.8" x2="55.88" y2="43.18" width="0.3048" layer="16"/>
+<wire x1="55.88" y1="50.8" x2="55.88" y2="36.195" width="0.3048" layer="16"/>
 </signal>
 <signal name="YELLOW">
 <contactref element="U1" pad="D4"/>
 <contactref element="LED" pad="2"/>
-<wire x1="53.34" y1="50.8" x2="53.34" y2="43.18" width="0.3048" layer="16"/>
+<wire x1="53.34" y1="50.8" x2="53.34" y2="36.195" width="0.3048" layer="16"/>
 </signal>
 <signal name="RED">
 <contactref element="U1" pad="D5"/>
 <contactref element="LED" pad="3"/>
-<wire x1="50.8" y1="50.8" x2="50.8" y2="43.18" width="0.3048" layer="16"/>
+<wire x1="50.8" y1="50.8" x2="50.8" y2="36.195" width="0.3048" layer="16"/>
 </signal>
 <signal name="5V">
@@
 <signal name="VIN">
 <contactref element="U1" pad="VIN"/>
-<contactref element="J1" pad="2"/>
+<contactref element="BATERRY" pad="2"/>
 <wire x1="45.72" y1="2.54" x2="45.72" y2="10.795" width="0.508" layer="1"/>
 <wire x1="45.72" y1="10.795" x2="40.64" y2="15.875" width="0.508" layer="1"/>
