File: PCB/ArduinoUnoCape/ArduinoCape.sch (EAGLE design)
At the start: 1 part, among them U1 ARDUINOR3-DIMENSION

Commit message: updated pcb and code
Parts:
- added 7-SEG-LED: 4P-2.0, Seeed-OPL-Connector:GROVE-CONNECTOR-DIP(4P-2.0)
- added BUTTON: (no value), pinhead:PINHD-1X2
- added J1: (no value), SparkFun-Connectors:CONN_02JST-PTH-2
- added LED: (no value), con-lstb:MA03-1
Connections:
- net 3V renamed 3V3
- new net VIN: J1.2, U1.VIN
- net 5V: now also 7-SEG-LED.3
- net BUTTON: now also BUTTON.2
- net GND: now also 7-SEG-LED.4, BUTTON.1, J1.1
- net GREEN: now also LED.1
- net RED: now also LED.3
- net SCL: now also 7-SEG-LED.1, U1.SCL; no longer U1.A5/SCL
- net SDA: now also 7-SEG-LED.2, U1.SDA; no longer U1.A4/SDA
- net YELLOW: now also LED.2
Changed lines of the file:
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@@
 <layer number="112" name="tSilk" color="7" fill="1" visible="no" active="yes"/>
 <layer number="113" name="ReferenceLS" color="7" fill="1" visible="no" active="no"/>
+<layer number="114" name="Badge_Outline" color="7" fill="1" visible="yes" active="yes"/>
+<layer number="115" name="ReferenceISLANDS" color="7" fill="1" visible="yes" active="yes"/>
 <layer number="116" name="Patch_BOT" color="9" fill="4" visible="no" active="yes"/>
+<layer number="117" name="BACKMAAT1" color="7" fill="1" visible="no" active="no"/>
 <layer number="118" name="Rect_Pads" color="7" fill="1" visible="no" active="no"/>
+<layer number="119" name="KAP_TEKEN" color="7" fill="1" visible="no" active="no"/>
+<layer number="120" name="KAP_MAAT1" color="7" fill="1" visible="no" active="no"/>
 <layer number="121" name="_tsilk" color="7" fill="1" visible="no" active="yes"/>
 <layer number="122" name="_bsilk" color="7" fill="1" visible="no" active="yes"/>
@@
 <layer number="128" name="_bValues" color="7" fill="1" visible="no" active="yes"/>
 <layer number="129" name="Mask" color="7" fill="1" visible="yes" active="yes"/>
+<layer number="130" name="SMDSTROOK" color="7" fill="1" visible="no" active="no"/>
 <layer number="131" name="tAdjust" color="7" fill="1" visible="no" active="yes"/>
 <layer number="132" name="bAdjust" color="7" fill="1" visible="no" active="yes"/>
+<layer number="133" name="bottom_silk" color="7" fill="1" visible="no" active="no"/>
 <layer number="144" name="Drill_legend" color="7" fill="1" visible="no" active="yes"/>
 <layer number="150" name="Notes" color="7" fill="1" visible="no" active="yes"/>
@@
 <parts>
 <part name="U1" library="adafruit" library_urn="urn:adsk.eagle:library:420" deviceset="ARDUINOR3" device="-DIMENSION"/>
+<part name="LED" library="con-lstb" library_urn="urn:adsk.eagle:library:162" deviceset="MA03-1" device=""/>
+<part name="7-SEG-LED" library="Seeed-OPL-Connector" deviceset="GROVE-CONNECTOR-DIP(4P-2.0)" device="" value="4P-2.0"/>
+<part name="J1" library="SparkFun-Connectors" deviceset="CONN_02" device="JST-PTH-2"/>
+<part name="BUTTON" library="pinhead" library_urn="urn:adsk.eagle:library:325" deviceset="PINHD-1X2" device=""/>
 </parts>
 <sheets>
@@
 <instances>
 <instance part="U1" gate="G$1" x="40.64" y="48.26" rot="R90"/>
+<instance part="LED" gate="G$1" x="96.52" y="48.26"/>
+<instance part="7-SEG-LED" gate="G$1" x="99.06" y="67.31" rot="R180"/>
+<instance part="J1" gate="G$1" x="96.52" y="25.4"/>
+<instance part="BUTTON" gate="G$1" x="96.52" y="83.82" rot="R180"/>
 </instances>
 <busses>
@@
 <net name="SCL" class="0">
 <segment>
-<pinref part="U1" gate="G$1" pin="A5/SCL"/>
-<wire x1="71.12" y1="71.12" x2="76.2" y2="71.12" width="0.1524" layer="91"/>
-<label x="73.66" y="71.12" size="1.778" layer="95"/>
+<pinref part="U1" gate="G$1" pin="SCL"/>
+<wire x1="10.16" y1="22.86" x2="5.08" y2="22.86" width="0.1524" layer="91"/>
+<label x="5.08" y="22.86" size="1.778" layer="95"/>
+</segment>
+<segment>
+<pinref part="7-SEG-LED" gate="G$1" pin="1"/>
+<wire x1="102.87" y1="63.5" x2="107.95" y2="63.5" width="0.1524" layer="91"/>
+<label x="105.41" y="63.5" size="1.778" layer="95"/>
 </segment>
 </net>
 <net name="SDA" class="0">
 <segment>
-<pinref part="U1" gate="G$1" pin="A4/SDA"/>
-<wire x1="71.12" y1="68.58" x2="76.2" y2="68.58" width="0.1524" layer="91"/>
-<label x="73.66" y="68.58" size="1.778" layer="95"/>
+<pinref part="U1" gate="G$1" pin="SDA"/>
+<wire x1="10.16" y1="25.4" x2="5.08" y2="25.4" width="0.1524" layer="91"/>
+<label x="5.08" y="25.4" size="1.778" layer="95"/>
+</segment>
+<segment>
+<pinref part="7-SEG-LED" gate="G$1" pin="2"/>
+<wire x1="102.87" y1="66.04" x2="107.95" y2="66.04" width="0.1524" layer="91"/>
+<label x="105.41" y="66.04" size="1.778" layer="95"/>
 </segment>
 </net>
@@
 <label x="5.08" y="63.5" size="1.778" layer="95"/>
 </segment>
+<segment>
+<pinref part="BUTTON" gate="G$1" pin="2"/>
+<wire x1="99.06" y1="83.82" x2="109.22" y2="83.82" width="0.1524" layer="91"/>
+<label x="106.68" y="83.82" size="1.778" layer="95"/>
+</segment>
 </net>
 <net name="GREEN" class="0">
@@
 <label x="5.08" y="60.96" size="1.778" layer="95"/>
 </segment>
+<segment>
+<pinref part="LED" gate="G$1" pin="1"/>
+<wire x1="104.14" y1="45.72" x2="109.22" y2="45.72" width="0.1524" layer="91"/>
+<label x="106.68" y="45.72" size="1.778" layer="95"/>
+</segment>
 </net>
 <net name="YELLOW" class="0">
@@
 <label x="5.08" y="58.42" size="1.778" layer="95"/>
 </segment>
+<segment>
+<pinref part="LED" gate="G$1" pin="2"/>
+<wire x1="104.14" y1="48.26" x2="109.22" y2="48.26" width="0.1524" layer="91"/>
+<label x="106.68" y="48.26" size="1.778" layer="95"/>
+</segment>
 </net>
 <net name="RED" class="0">
@@
 <label x="5.08" y="55.88" size="1.778" layer="95"/>
 </segment>
+<segment>
+<pinref part="LED" gate="G$1" pin="3"/>
+<wire x1="104.14" y1="50.8" x2="109.22" y2="50.8" width="0.1524" layer="91"/>
+<label x="106.68" y="50.8" size="1.778" layer="95"/>
+</segment>
 </net>
 <net name="GND" class="0">
@@
 <label x="73.66" y="50.8" size="1.778" layer="95"/>
 </segment>
+<segment>
+<pinref part="7-SEG-LED" gate="G$1" pin="4"/>
+<wire x1="102.87" y1="71.12" x2="107.95" y2="71.12" width="0.1524" layer="91"/>
+<label x="105.41" y="71.12" size="1.778" layer="95"/>
+</segment>
+<segment>
+<pinref part="J1" gate="G$1" pin="1"/>
+<wire x1="104.14" y1="25.4" x2="109.22" y2="25.4" width="0.1524" layer="91"/>
+<label x="106.68" y="25.4" size="1.778" layer="95"/>
+</segment>
+<segment>
+<pinref part="BUTTON" gate="G$1" pin="1"/>
+<wire x1="99.06" y1="81.28" x2="109.22" y2="81.28" width="0.1524" layer="91"/>
+<label x="106.68" y="81.28" size="1.778" layer="95"/>
+</segment>
 </net>
 <net name="5V" class="0">
@@
 <label x="73.66" y="45.72" size="1.778" layer="95"/>
 </segment>
-</net>
-<net name="3V" class="0">
+<segment>
+<pinref part="7-SEG-LED" gate="G$1" pin="3"/>
+<wire x1="102.87" y1="68.58" x2="107.95" y2="68.58" width="0.1524" layer="91"/>
+<label x="105.41" y="68.58" size="1.778" layer="95"/>
+</segment>
+</net>
+<net name="3V3" class="0">
 <segment>
 <pinref part="U1" gate="G$1" pin="3V"/>
@@
 </segment>
 </net>
+<net name="VIN" class="0">
+<segment>
+<pinref part="U1" gate="G$1" pin="VIN"/>
+<wire x1="71.12" y1="53.34" x2="76.2" y2="53.34" width="0.1524" layer="91"/>
+<label x="73.66" y="53.34" size="1.778" layer="95"/>
+</segment>
+<segment>
+<pinref part="J1" gate="G$1" pin="2"/>
+<wire x1="104.14" y1="27.94" x2="109.22" y2="27.94" width="0.1524" layer="91"/>
+<label x="106.68" y="27.94" size="1.778" layer="95"/>
+</segment>
+</net>

Commit message: asdf
Parts:
- 7-SEG-LED: value 4P-2.0 -> (none)
- renumbered J1 to BATERRY
Changed lines of the file:
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@@
 <part name="U1" library="adafruit" library_urn="urn:adsk.eagle:library:420" deviceset="ARDUINOR3" device="-DIMENSION"/>
 <part name="LED" library="con-lstb" library_urn="urn:adsk.eagle:library:162" deviceset="MA03-1" device=""/>
-<part name="7-SEG-LED" library="Seeed-OPL-Connector" deviceset="GROVE-CONNECTOR-DIP(4P-2.0)" device="" value="4P-2.0"/>
-<part name="J1" library="SparkFun-Connectors" deviceset="CONN_02" device="JST-PTH-2"/>
+<part name="7-SEG-LED" library="Seeed-OPL-Connector" deviceset="GROVE-CONNECTOR-DIP(4P-2.0)" device=""/>
+<part name="BATERRY" library="SparkFun-Connectors" deviceset="CONN_02" device="JST-PTH-2"/>
 <part name="BUTTON" library="pinhead" library_urn="urn:adsk.eagle:library:325" deviceset="PINHD-1X2" device=""/>
 </parts>
@@
 <instance part="LED" gate="G$1" x="96.52" y="48.26"/>
 <instance part="7-SEG-LED" gate="G$1" x="99.06" y="67.31" rot="R180"/>
-<instance part="J1" gate="G$1" x="96.52" y="25.4"/>
+<instance part="BATERRY" gate="G$1" x="96.52" y="25.4"/>
 <instance part="BUTTON" gate="G$1" x="96.52" y="83.82" rot="R180"/>
 </instances>
@@
 </segment>
 <segment>
-<pinref part="J1" gate="G$1" pin="1"/>
+<pinref part="BATERRY" gate="G$1" pin="1"/>
 <wire x1="104.14" y1="25.4" x2="109.22" y2="25.4" width="0.1524" layer="91"/>
 <label x="106.68" y="25.4" size="1.778" layer="95"/>
@@
 </segment>
 <segment>
-<pinref part="J1" gate="G$1" pin="2"/>
+<pinref part="BATERRY" gate="G$1" pin="2"/>
 <wire x1="104.14" y1="27.94" x2="109.22" y2="27.94" width="0.1524" layer="91"/>
 <label x="106.68" y="27.94" size="1.778" layer="95"/>
